File: TransceiverPCB/TransceiverPCB.kicad_sch (KiCad schematic)
At the start: 65 parts, among them IC1 QPL6220QTR7, IC2 AD9218BSTZ-65, IC3 AD9763ASTZ, IC4 ADF4351BCPZ-RL7, J1 USB4085-GF-A_REVB, J2 RFPC-SMA27-F, J3 RFPC-SMA27-F, SW1 SW_Push, SW2 SW_Push, U1 XC7A35T-1FTG256C, U10 AP2112K-3.3TRG1, U11 LM66100DCKR, U12 ADL5387ACPZ-R7, U2 W25Q32JVSSIQ, U3 W25Q32JVSSIQ, U4 DSC1001CI2-100.0000T, U6 ADL5375-05ACPZ-R7, U7 ADA4940-2ACPZ-R7, U8 ADL5320ARKZ-R7, U9 SC09147, X1 ABM8-272-T3

Commit message: Connected demod to FDA to LPF
- connected BPF to demod with balun
- connected demod to FDA, still need to establish Vocm
- FDA output to LPF corner freq. 1.9 MHz
- connected REFOUT of ADC to pin 4, indicating Vpp of 2V and output data using two's complement
Parts:
- added C31, C32, C33, C34: 10uF, symbol Device:C
- added C38, C39: 270pF, symbol Device:C
- added C40, C41: 91pF, symbol Device:C
- added C42, C43: 68pF, symbol Device:C
- added C46, C47, C50, C52: .1uF, symbol Device:C
- added C48, C49, C51: 100pF, symbol Device:C
- added C53, C54: 1000pF, symbol Device:C
- added L10, L13, L4, L5, L6, L7, L8, L9: 27uH, symbol Device:L
- added L11, L12, L14, L15: 10uH, symbol Device:L
- added L2, L3: 120nH, symbol Device:L
- added R11, R12: 500, symbol Device:R_US
- added R13, R20, R21, R22, R23, R24, R25, R26: 1k, symbol Device:R_US
- added T1: ETC1-1-13TR, ETC1-1-13TR_MCM, symbol LIB_IRISHSAT:ETC1-1-13TR
Connections:
- net +5V: now also U12.1 (VPA), U12.17 (VPB), U12.18 (VPB), U12.19 (VPX), U12.4 (VPL), U12.5 (VPL), U12.6 (VPL), C46.1, C47.1, C48.1, C49.1, C50.1, C51.1
- net DEMOD_RF_IN: now also T1.2
- net GND: now also U12.10 (CML), U12.11 (CML), U12.12 (COM), U12.2 (COM), U12.20 (CMRF), U12.23 (CMRF), U12.24 (CMRF), U12.25 (GND), U12.7 (CML), U7.15 (VS2-), U7.21 (VS1-), U7.22 (VS1-), U7.HTAB (EPAD), C46.2, C47.2, C48.2, C49.2, C50.2, C51.2, C52.1, L2.1, L3.2, T1.1
- net IN1-: now reaches U7.1 (IN1-)
- net IN1-: now also R21.2, R24.1
- net ADC_Vocm: now reaches U7.11 (VOCM2)
- net ADC_Vocm: now also U7.17 (VOCM1)
- net IOUT+: now reaches U7.12 (OUT2+)
- net IOUT+: now also C33.1
- net IOUT-: now reaches U7.13 (OUT2-)
- net IOUT-: now also C34.1
- net QOUT+: now reaches U7.18 (OUT1+)
- net QOUT+: now also C31.1
- net QOUT-: now reaches U7.19 (OUT1-)
- net QOUT-: now also C32.1
- net at U7.2 (FB1+): now also R24.2
- net at U7.23 (FB1-): now also R13.1
- net IN1+: now reaches U7.24 (IN1+)
- net IN1+: now also R13.2, R20.2
- net at U7.5 (FB2-): now also R25.2
- net IN2+: now reaches U7.6 (IN2+)
- net IN2+: now also R22.2, R25.1
- net IN2-: now reaches U7.7 (IN2-)
- net IN2-: now also R23.2, R26.1
- net at U7.8 (FB2+): now also R26.2
- net at IC2.4 (DFS/GAIN): now also IC2.6 (REFOUT), C52.2
- net at U12.13 (ILO): now also R23.1
- net at U12.14 (IHI): now also R22.1
- net at U12.15 (QLO): now also R21.1
- net at U12.16 (QHI): now also R20.1
- net RFIN: now reaches U12.21 (RFIN)
- net RFIN: now also C53.1, L3.1
- net RFIP: now reaches U12.22 (RFIP)
- net RFIP: now also C54.1, L2.2
- new net: C38.1, L13.1, L8.2
- new net: C40.1, L13.2, L14.1
- new net: C41.1, L10.2, L12.1
- new net: C41.2, L11.1, L6.2
- new net: C39.2, L4.2, L6.1
- new net: C31.2, L8.1
- new net: C32.2, L5.1
- new net: C38.2, L5.2, L9.1
- new net: C39.1, L10.1, L7.2
- new net: C40.2, L15.1, L9.2
- new net: C53.2, T1.5
- new net: C54.2, T1.3
- new net: C33.2, L7.1
- new net: C34.2, L4.1
- new net IHI: C43.1, L12.2, R12.1
- new net ILO: C43.2, L11.2, R12.2
- new net QHI: C42.1, L14.2, R11.1
- new net QLO: C42.2, L15.2, R11.2
Other:
- note added: "1.9 MHz LPF MOD OUTPUT TO ADC"
- note added: "Pin4 -> REFOUT indicates 2s complement and 2Vpp"
- note added: "power bypass capacitors must be electrically as close as possible"
- note removed: "Needs a balun"
- moved on the sheet: C3, C4, FL2, FL4, IC1, IC2, J3, U12, U7

Commit message: Added some images and comments
Parts:
- removed FL3: B39921B2672P810, B39921B2672P810, symbol LIB_IRISHSAT:B39921B2672P810
- added C30, C35: 100nF, symbol Device:C
Connections:
- net ADC_Vocm is gone; now on net +1V1: U7.11 (VOCM2), U7.17 (VOCM1)
- net +1V1: now also C30.2, C35.2
- net GND: now also C30.1, C35.1
Other:
- moved on the sheet: C31, C32, C33, C34, C38, C39, C40, C41, C42, C43, FL1, J2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

Commit message: LO Connections
-Connected LO to RP2040
-Connected to power
-Decoupled

-Looking into loop filter
Parts:
- added C36, C37, C45, C55, C56: 1uF, symbol Device:C
- added C44: C, symbol Device:C
Connections:
- net GND: now also IC4.11 (AGNDVCO_1), IC4.18 (AGNDVCO_2), IC4.21 (AGNDVCO_3), IC4.27 (DGND), IC4.31 (SDGND), IC4.33 (EXPOSED_PAD_(GND)), IC4.9 (AGND), C36.1, C37.2, C45.1, C55.2, C56.2
- net CLK_ADF4351_LO: now reaches IC4.1 (CLK)
- net CLK_ADF4351_LO: now also U9.13 (GPIO10)
- net +3.3V: now reaches IC4.10 (AVDD)
- net +3.3V: now also IC4.16 (VVCO_1), IC4.17 (VVCO_2), IC4.28 (DVDD), IC4.32 (SDVDD), IC4.6 (VP), C36.2, C37.1, C44.1, C45.2, C55.1, C56.1
- net DATA_ADF4351_LO: now reaches IC4.2 (DATA)
- net DATA_ADF4351_LO: now also U9.14 (GPIO11)
- net LD_ADF4351_LO: now reaches IC4.25 (LD)
- net LD_ADF4351_LO: now also U9.17 (GPIO14)
- net LE_ADF4351_LO: now reaches IC4.3 (LE)
- net LE_ADF4351_LO: now also U9.15 (GPIO12)
- net CE_ADF4351_LO: now reaches IC4.4 (CE)
- net CE_ADF4351_LO: now also U9.16 (GPIO13)
- no-connect marks 43 -> 38
Other:
- note added: "Need to look into loop filter mentioned in data sheet for pins 5, 7, and 8"
- note added: "Suuuuuuure suuuuuuure"

Commit message: Modulator and Power Amplifier Complete
Completed mod and PA
Might need to change LO input and DAC filter - review changes
Parts:
- added C57, C62: 47pF, symbol Device:C
- added C58: 6.8pF, symbol Device:C
- added C59: 100pF, symbol Device:C
- added C60: 10nF, symbol Device:C
- added C61: 10uF, symbol Device:C
- added C63: 2.2pF, symbol Device:C
- added C64, C66: 53.62pF, symbol Device:C
- added C65, C67: 350.1pF, symbol Device:C
- added L16: 47nH, symbol Device:L
- added L17, L18, L19, L20: 771.1nH, symbol Device:L
- added R1, R14, R16, R17: 50, symbol Device:R_US
- added R15, R18: 100, symbol Device:R_US
Connections:
- net +5V: now also C59.1, C60.1, C61.1, L16.1
- net GND: now also C5.1, C6.1, C7.2, C8.2, C58.2, C59.2, C60.2, C61.2, C63.2, R1.2, R14.1, R16.2, R17.1
- net MOD_OUT: now also C57.1
- net PA_IN: now also C57.2, C58.1
- net PA_OUT: now also C62.2; no longer U8.3 (RFOUT)
- net QBBP: now reaches U6.10 (QBBP)
- net QBBP: now also C67.2, L20.2, R18.2
- net IBBP: now reaches U6.21 (IBBP)
- net IBBP: now also C65.1, L17.2, R15.1
- net IBBN: now reaches U6.22 (IBBN)
- net IBBN: now also C65.2, L18.2, R15.2
- net QBBN: now reaches U6.9 (QBBN)
- net QBBN: now also C67.1, L19.2, R18.1
- net IOUTA2: now reaches IC3.39 (IOUTA2)
- net IOUTA2: now also C66.2, L20.1, R17.2
- net IOUTB2: now reaches IC3.40 (IOUTB2)
- net IOUTB2: now also C66.1, L19.1, R16.1
- net IOUTB1: now reaches IC3.45 (IOUTB1)
- net IOUTB1: now also C64.2, L18.1, R14.2
- net IOUTA1: now reaches IC3.46 (IOUTA1)
- net IOUTA1: now also C64.1, L17.1, R1.1
- new net: C62.1, C63.1, L16.2, U8.3 (RFOUT)
Other:
- note added: "100 mils"
- note added: "200 mils"
- note added: "350 mils"
- note added: "75 mils"
- note added: "Line must be 200 mils after C58"
- note removed: "LPF"
- moved on the sheet: IC3, U8

Commit message: Added some comments, power rail for modulator
Parts:
- C44: value C -> 1uF
Connections:
- net +3.3V: now also C44.2; no longer C44.1
- net +5V: now also C5.2, C6.2, C7.1, C8.1, U6.18 (VPS1), U6.24 (VPS2)
- net GND: now also C44.1
- net IN1+ renamed DEMOD_IN1+
- net IN1- renamed DEMOD_IN1-
- net IN2+ renamed DEMOD_IN2+
- net IN2- renamed DEMOD_IN2-
- net RFIN renamed DEMOD_RFIN
- net RFIP renamed DEMOD_RFIP
Other:
- note added: "2xLO Frequency"
- note added: "9 Thermal Vias to GND"
- note added: "?"
- moved on the sheet: C3, C37, C4, C44, C46, C47, C48, C49, C50, C51, C53, C54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

Commit message: FPGA
- added 1.8V LDO
- added 1.0V LDO
- VCCO pins on FPGA
- QSPI Flash memory for FPGA
- Oscillator for FPGA
- Lots of decoupling capacitors
- Lots of VCC pins on teh FPGA
Parts:
- added C100, C103, C104, C99: 1uF, symbol Device:C
- added C101, C105, C75: 0.1uF, symbol Device:C
- added C102, C106: 10uF, symbol Device:C
- added C107, C108, C109, C110, C111, C112, C113, C114, C68, C69, C70, C71, C72, C73, C76, C77, C78, C79, C80, C81, C82, C83, C84, C85, C86, C87, C88, C89, C90, C91, C92, C93, C94, C95, C96, C97: 100nF, symbol Device:C
- added C74, C98: 4.7uF, symbol Device:C
- added D2, D3: LED, symbol Device:LED
- added J4: FPGA JTAG, Connector_IDC:IDC-Header_2x03_P2.54mm_Vertical_SMD, symbol Connector_Generic:Conn_02x03_Odd_Even
- added R19, R27, R28, R31, R32: 10k, symbol Device:R_US
- added R29: 1k, symbol Device:R_US
- added R30: DNF, symbol Device:R_US
- added SW3, SW4: SW_Push, symbol Switch:SW_Push
- added U13: LP5912-1.0DRVR, LIB_IRISHSAT:DRV0006A-IPC_A, symbol LIB_IRISHSAT:LP5912-1.0DRVR
- added U5: AP2112K-1.8TRG1, LIB_IRISHSAT:AP2112K-1.8TRG1_DIO, symbol LIB_IRISHSAT:AP2112K-1.8TRG1
- FL1, FL4: footprint B39921B2672P810 -> LIB_IRISHSAT:B39921B2672P810
- IC1: footprint SON50P200X200X90-9N-D -> LIB_IRISHSAT:SON50P200X200X90-9N-D
- IC2, IC3: footprint QFP50P900X900X160-48N -> LIB_IRISHSAT:QFP50P900X900X160-48N
- IC4: footprint QFN50P500X500X80-33N-D -> LIB_IRISHSAT:QFN50P500X500X80-33N-D
- T1: footprint ETC1-1-13TR_MCM -> LIB_IRISHSAT:ETC1-1-13TR_MCM
- U1: footprint FT/FTG256ARTIX-7_AMD -> LIB_IRISHSAT:FT&slash_FTG256ARTIX-7_AMD
- U10: footprint SOT_RG1_DIO -> LIB_IRISHSAT:SOT_RG1_DIO
- U11: footprint DCK6_TEX -> LIB_IRISHSAT:DCK6_TEX
- U12: footprint CP-24-14_ADI -> LIB_IRISHSAT:CP-24-14_ADI
- U2, U3: footprint SOIC-8_5P28X5P28_WIN -> LIB_IRISHSAT:SOIC-8_5P28X5P28_WIN
- U4: footprint CDFN4_3P2X2P5_MCH -> LIB_IRISHSAT:CDFN4_3P2X2P5_MCH
- U6, U7: footprint CP_24_7_ADI -> LIB_IRISHSAT:CP_24_7_ADI
- U8: footprint RK_3_ADI -> LIB_IRISHSAT:RK_3_ADI
- U9: footprint QFN56_7X7_RPI -> LIB_IRISHSAT:QFN56_7X7_RPI
- X1: footprint ABM8-272-T3_ABR -> LIB_IRISHSAT:ABM8-272-T3_ABR
Connections:
- net +1V1: no longer C21.2, C22.2, C23.2, U9.23 (DVDD), U9.45 (VREG_VOUT), U9.50 (DVDD)
- net +3V3: now also U1.A16 (VCCO_15), U1.A6 (VCCO_35), U1.B13 (VCCO_15), U1.B3 (VCCO_35), U1.C10 (VCCO_15), U1.D7 (VCCO_35), U1.E14 (VCCO_15), U1.E3 (IO_L11P_T1_SRCC_35), U1.F1 (VCCO_35), U1.H15 (VCCO_15), U1.J12 (VCCO_15), U1.J2 (VCCO_35), U1.L16 (VCCO_14), U1.L6 (VCCO_0), U1.M13 (VCCO_14), U1.M3 (VCCO_34), U1.N10 (VCCO_14), U1.R14 (VCCO_14), U1.R4 (VCCO_34), U1.T1 (VCCO_34), U2.8 (VCC), U4.1 (*STANDBY), U4.4 (VDD), C68.1, C69.1, C70.2, C71.1, C72.1, C73.1, C74.1, C75.1, C76.1, C77.1, C78.1, C79.1, C80.1, C81.1, C82.1, C83.1, C84.1, C85.1, C86.1, C87.1, C88.1, C89.1, C90.1, C91.1, C92.1, D2.1 (K), D3.1 (K), J4.2 (VREF), R28.2, R30.1
- net +5V: now also C25.1, C26.2, C27.2, R10.1, U10.1 (VIN), U11.6 (VOUT), C103.2, C99.2, R31.1, R32.1, U13.6 (IN), U5.1 (VIN); no longer C12.2, D1.2 (C), J1.A4 (VBUS), J1.A9 (VBUS__1), J1.B4 (VBUS__2), J1.B9 (VBUS__3), L1.2
- net GND: now also C25.2, U1.J11 (GND), U1.J9 (GND), U1.K14 (GND), U2.4 (GND), U4.2 (GND), C100.1, C101.1, C102.1, C103.1, C104.1, C105.1, C106.1, C107.2, C108.2, C109.2, C110.2, C111.2, C112.2, C113.2, C114.2, C68.2, C69.2, C70.1, C71.2, C72.2, C73.2, C74.2, C75.2, C76.2, C77.2, C78.2, C79.2, C80.2, C81.2, C82.2, C83.2, C84.2, C85.2, C86.2, C87.2, C88.2, C89.2, C90.2, C91.2, C92.2, C93.2, C94.2, C95.2, C96.2, C97.2, C98.2, C99.1, J4.6 (GND), SW3.2, SW4.1, U13.5 (GND), U13.7 (Thermal_Pad), U5.2 (GND); no longer C25.1
- net USB_BOOT: now also R29.2, SW4.2
- net +1V: now reaches U1.F11 (VCCBRAM)
- net +1V: now also U1.E10 (VCCBRAM), U1.F7 (VCCINT), U1.F9 (VCCINT), U1.G6 (VCCINT), U1.H9 (VCCINT), U1.J6 (VCCINT), U1.K9 (VCCINT), U1.L8 (VCCINT), C104.2, C105.2, C106.2, C107.1, C108.1, C109.1, C110.1, C111.1, C112.1, C113.1, C114.1, C93.1, U13.1 (OUT)
- net +1V8: now reaches U1.G10 (VCCAUX)
- net +1V8: now also U1.J10 (VCCAUX), U1.K11 (VCCAUX), U1.L10 (VCCAUX), C100.2, C101.2, C102.2, C94.1, C95.1, C96.1, C97.1, C98.1, U5.5 (VOUT)
- net at U1.H10 (DONE_0): now also R27.1
- net QSPI_SD1_FPGA: now reaches U1.J14 (IO_L1N_T0_D01_DIN_14)
- net QSPI_SD1_FPGA: now also U2.2 (DO(IO1))
- net at U1.K10 (INIT_B_0): now also R19.1
- net QSPI_SD2_FPGA: now reaches U1.K15 (IO_L2P_T0_D02_14)
- net QSPI_SD2_FPGA: now also U2.3 (/WP(IO2))
- net QSPI_SD3_FGPA: now reaches U1.K16 (IO_L2N_T0_D03_14)
- net QSPI_SD3_FGPA: now also U2.7 (/HOLD_OR_/RESET(IO3))
- net FPGA_TCK: now reaches U1.L7 (TCK_0)
- net FPGA_TCK: now also J4.3 (TCK)
- net at U1.L9 (PROGRAM_B_0): now also R28.1, SW3.1
- net FPGA_OSCILLATOR_100MHZ: now reaches U4.3 (OUT)
- net FPGA_OSCILLATOR_100MHZ: now also U1.P10 (IO_L14P_T2_SRCC_14)
- net QSPI_SS_FPGA: now reaches U2.1 (/CS)
- net QSPI_SS_FPGA: now also U1.R13 (IO_L16P_T2_CSI_B_14), R29.1, R30.2
- net QSPI_SD0_FPGA: now reaches U2.5 (DI(IO0))
- net QSPI_SD0_FPGA: now also U1.T12 (IO_L15N_T2_DQS_DOUT_CSO_B_14)
- net QSPI_SCLK_FPGA: now reaches U2.6 (CLK)
- net QSPI_SCLK_FPGA: now also U1.E8 (CCLK_0)
- net FPGA_TMS: now reaches U1.M7 (TMS_0)
- net FPGA_TMS: now also J4.1 (TMS)
- net FPGA_TDI: now reaches U1.N7 (TDI_0)
- net FPGA_TDI: now also J4.5 (TDI)
- net FPGA_TDO: now reaches U1.N8 (TDO_0)
- net FPGA_TDO: now also J4.4 (TDO)
- new net: D2.2 (A), R19.2
- new net: C12.2, D1.2 (C), J1.A4 (VBUS), J1.A9 (VBUS__1), J1.B4 (VBUS__2), J1.B9 (VBUS__3), L1.2
- new net: R32.2, U13.4 (EN)
- new net: D3.2 (A), R27.2
- new net: R31.2, U5.3 (EN)
- new net +1V1_RP2040_INTERNAL: C21.2, C22.2, C23.2, U9.23 (DVDD), U9.45 (VREG_VOUT), U9.50 (DVDD)
- no-connect marks 38 -> 41
Other:
- note added: "1-2cm from FPGA"
- note added: "Can we use the +1V rail instead of +1V1?????"
- note added: "Either 3A or 5A limit USB"
- note added: "Filtered 5V"
- note added: "JTAG Programmer"
- note added: "Maybe use a buck converter instead for +1V, +1V8, +1V1"
- note added: "POWER AND USB"
- note added: "Place as close as possible to FPGA"
- note added: "RP2040"
- note added: "This is +5V but not too clean"
- note added: "USB to +1V"
- note added: "USB to +1V8"
- note added: "USB to +3V3"
- note removed: "Decoupling C?"
- note removed: "USB to 3.3V with Filters and Protection"
- moved on the sheet: C1, C10, C11, C12, C13, C14, C15, C16, C17, C18, C19, C2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

Commit message: Filter LO to DAC, ADC/DAC power pins
Created filter from LO to DAC
Wired ADC and DAC power pins
Parts:
- added C115, C117: 120pF, symbol Device:C
- added C116, C121, C122, C123, C129, C130, C131, C132, C133, C134, C135: 0.1uF, symbol Device:C
- added C118, C120, C124, C126: 3.3pF, symbol Device:C
- added C119, C125: 4.7pF, symbol Device:C
- added C127, C128: 1nF, symbol Device:C
- added L21, L22, L23, L24: 2.7nH, symbol Device:L
- added L25, L26: 19nH, symbol Device:L
- added R33: 100, symbol Device:R_US
- C1, C2: value 100pF -> 0.1uF
Connections:
- net +1V1 is gone; now on net +1V: C30.2, C35.2, U7.11 (VOCM2), U7.17 (VOCM1)
- net IHI is gone; now on net I+ADC_IN: C43.1, L12.2, R12.1
- net ILO is gone; now on net I-ADC_IN: C43.2, L11.2, R12.2
- net QHI is gone; now on net Q+ADC_IN: C42.1, L14.2, R11.1
- net QLO is gone; now on net Q-ADC_IN: C42.2, L15.2, R11.2
- net +3V3: now also C1.1, C2.1, IC2.15 (VDD_1), IC2.28 (VDD_2), IC2.33 (VDD_3), IC2.46 (VDD_4), IC3.16 (DVDD1), IC3.22 (DVDD2), IC3.47 (AVDD), IC3.48 (MODE), C115.1, C116.1, C117.1, C121.1, C122.1, C133.1, C134.1, C135.1, L25.1, L26.1
- net +5V: now also U7.10 (VS2+), U7.16 (VS2+), U7.3 (VS1+), U7.4 (VS1+), U7.9 (VS2+)
- net GND: now also C1.2, C2.2, IC2.9 (S2), IC3.15 (DCOM1), IC3.21 (DCOM2), IC3.38 (ACOM), C115.2, C116.2, C117.2, C118.1, C119.1, C120.1, C121.2, C122.2, C123.2, C124.2, C125.2, C126.2, C129.2, C130.2, C131.2, C132.2, C133.2, C134.2, C135.2
- net LO_A_OUT+: now also C118.2, L21.2, L25.2, R33.1; no longer C1.1
- net LO_A_OUT-: now also C124.1, L23.2, L26.2, R33.2; no longer C2.1
- net LOIN_mod: now reaches U6.4 (LOIN)
- net LOIN_mod: now also C127.2; no longer C2.2
- net Q-ADC_IN: now reaches IC2.10 (~{AINB})
- net Q+ADC_IN: now reaches IC2.11 (AINB)
- net +3V: now reaches IC2.13 (VD_1)
- net +3V: now also IC2.30 (VD_2), IC2.31 (VD_3), IC2.48 (VD_4), IC2.8 (S1), C123.1, C129.1, C130.1, C131.1, C132.1
- net I+ADC_IN: now reaches IC2.2 (AINA)
- net I-ADC_IN: now reaches IC2.3 (~{AINA})
- net LOIP_mod: now reaches U6.3 (LOIP)
- net LOIP_mod: now also C128.2; no longer C1.2
- new net: C120.2, C128.1, L22.1
- new net: C119.2, L21.1, L22.2
- new net: C125.1, L23.1, L24.2
- new net: C126.1, C127.1, L24.1
- no-connect marks 41 -> 44
Other:
- note added: "3rd harmonic filter, LO output to modulator"
- note added: "?????????????????"
- note added: "Can we use the +1V rail instead of +1V1????? Sure"
- note added: "Disable pin able to be left floating due to internal pull up network"
- note added: "Note: potentially use voltage divider if not much current is needed for odd voltage levels"
- moved on the sheet: C5, C52, C55, C6, C64, C65, C66, C67, C7, C8, IC2, IC3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
