File: TransceiverPCB/TransceiverPCB.kicad_pcb (KiCad board)
At the start: 6 copper layers, 296 parts, among them IC1 QPL6220QTR7, IC2 AD9218BSTZ-65, IC3 AD9763ASTZ, IC4 ADF4351BCPZ-RL7, J1 USB4085-GF-A_REVB, J2 RFPC-SMA27-F, J3 RFPC-SMA27-F, J5 Conn_01x02, J6 878321420, Q1 AO3401A, Q2 AO3401A, SW1 SW_Push, SW2 SW_Push, SW4 SW_Push, T1 ETC1-1-13TR, U1 XC7A35T-1FTG256C, U10 AP2112K-3.3TRG1, U11 TPS62840DLCR, U12 ADL5387ACPZ-R7, U13 TPS62933FDRLR, U14 DSC1001CI2-100.0000T, U15 TPS62840DLCR, U16 TPS62841DLCR, U2 W25Q32JVSSIQ, U3 W25Q32JVSSIQ, U4 DSC1001CI2-100.0000T, U5 LTC4412ES6-TRMPBF, U6 ADL5375-05ACPZ-R7, U7 ADA4940-2ACPZ-R7, U8 ADL5320ARKZ-R7, U9 SC09147, X1 ABM8-272-T3

Commit message: First Draft of PCB
Its pretty bad (oh well)
Parts:
- moved C36 234.2 mm to (138.4, 111.9), turned to 90 degrees
- moved C90 233.3 mm to (135.8, 107.4), turned to 180 degrees
- moved C44 229.5 mm to (143.4, 112.0), turned to 90 degrees
- moved C87 229.3 mm to (146.4, 109.2)
- moved C45 224.8 mm to (146.4, 110.8), turned to 180 degrees
- moved C86 224.6 mm to (146.1, 107.9)
- moved C55 220.2 mm to (141.6, 100.9), turned to 90 degrees
- moved C56 220.1 mm to (139.3, 101.7), turned to 90 degrees
- moved C88 219.6 mm to (144.0, 102.2), turned to 90 degrees
- moved C89 218.3 mm to (148.0, 99.6)
- moved R55 217.6 mm to (147.7, 104.7)
- moved IC4 217.3 mm to (141.0, 106.5), turned to 0 degrees
- moved C145 212.8 mm to (150.8, 118.8), turned to -90 degrees
- moved C144 212.3 mm to (153.0, 117.6), turned to -90 degrees
- moved C155 212.1 mm to (147.8, 101.1)
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Connections:
- net FPGA_JTAG_VREF renamed +3V3
- R11 pad 1: /Q+ADC_IN -> /Q-ADC_IN
- R11 pad 2: /Q-ADC_IN -> /Q+ADC_IN
Routing:
- net LNA_ShutDown: track 0.00 -> 83.8 mm
- net /IOUTB2: track 0.00 -> 46.4 mm
- net /IOUTA2: track 0.00 -> 43.1 mm
- net +3V: track 4.39 -> 42.5 mm
- net /LO_A_OUT+: track 0.00 -> 34.0 mm, vias 0 -> 2
- net /VTUNE_ADF4351_LO: track 0.00 -> 29.1 mm
- net /DEMOD_IN2-: track 1.41 -> 30.5 mm, vias 0 -> 2
- net +5V: track 43.2 -> 71.7 mm
- net /DEMOD_IN2+: track 1.72 -> 26.7 mm, vias 0 -> 2
- net /DEMOD_IN1-: track 1.72 -> 22.8 mm, vias 0 -> 2
- net /LO_A_OUT-: track 0.00 -> 21.1 mm
- net /DEMOD_IN1+: track 2.13 -> 22.5 mm, vias 0 -> 2
- net /LO_B_OUT-: track 0.00 -> 19.8 mm
- net /LO_B_OUT+: track 0.00 -> 19.2 mm, vias 0 -> 2
- net /IOUT+: track 0.00 -> 18.8 mm, vias 0 -> 2
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Other:
- board text added: "Custon Transceiver Rylan Paul, Thomas Mancini, Caden Niziol, Joaquin Caraveo, Ana Arnett, Alyssa Riter"
- board text removed: "Best Case: Custom Transceiver Worst Case: Smoke Machine Rylan Paul, Thomas Mancini, Caden Niziol, Joaquin Caraveo, Ana Arnett, Alyssa Riter"
