File: IrishSat_Transceiver_I_Hardly_Know_Her/IrishSat_Transceiver_I_Hardly_Know_Her.kicad_sch (KiCad schematic)
At the start: 0 parts

Commit message: Created Power Amplifier
QPA9127 integration
Parts:
- added C1: 0.1u, Package_SO:SOIC-8_3.9x4.9mm_P1.27mm, symbol Device:C
- added C2: 1000p, Package_SO:SOIC-8_3.9x4.9mm_P1.27mm, symbol Device:C
- added C3, C4: 10p, Package_SO:SOIC-8_3.9x4.9mm_P1.27mm, symbol Device:C
- added L1: 12n, symbol Device:L
- added R1: 220k, symbol Device:R_US
- added U1: QPA9127, DFN8_2X2_QOR, symbol LIB_IRISHSAT:QPA9127
Connections:
- new net: C3.1, L1.2, U1.7 (RFOUT)
- new net: C4.2, U1.2 (RFIN)
- new net +5V: C1.1, C2.1, L1.1
- new net GND: C1.2, C2.2, R1.2, U1.4 (GND), U1.6 (GND), U1.9 (RF/DC_GND)
- new net PA_SHUT_DOWN: R1.1, U1.5 (SHUT_DOWN)
- new net RF_IN: C4.1
- new net RF_OUT: C3.2
